File: powerbank_pcb/powerbank_pcb.kicad_pcb (KiCad board)
At the start: 2 copper layers, 18 parts, among them SW1 TS-1101-C-W, U1 TP4366E

Commit message: update
Parts:
- moved USB1 68.0 mm to (112.5, 71.3), turned to -90 degrees
- moved U1 61.1 mm to (128.5, 70.9), turned to 180 degrees
- moved L1 55.2 mm to (124.5, 63.0), turned to 180 degrees
- moved R2 50.8 mm to (119.0, 68.5), turned to 90 degrees
- moved R1 50.0 mm to (119.0, 74.0), turned to -90 degrees
- moved C3 38.1 mm to (131.0, 65.5)
- moved C1 37.0 mm to (133.0, 69.5), turned to 90 degrees
- moved C2 33.9 mm to (135.5, 69.5), turned to 90 degrees
- moved C4 13.1 mm to (156.0, 71.7)
- moved R3 13.1 mm to (156.0, 81.6)
- moved R4 13.1 mm to (156.0, 84.9)
Routing:
- net GND: track 0.00 -> 24.3 mm
- net Vin: track 0.00 -> 19.5 mm
- net Net-(U1-SW): track 0.00 -> 8.46 mm
- net Vout: track 0.00 -> 7.63 mm
- net Bat: track 0.00 -> 6.05 mm
- net Net-(USB1-CC1): track 0.00 -> 4.83 mm
- net Net-(USB1-CC2): track 0.00 -> 4.79 mm

Commit message: update
Parts:
- moved SW1 57.5 mm to (142.0, 76.5), turned to 180 degrees
- moved D5 51.4 mm to (122.8, 76.5)
- moved BT1 37.7 mm to (143.0, 61.0)
- moved D1 32.5 mm to (142.8, 71.2), turned to 180 degrees
- moved D2 31.4 mm to (142.8, 69.5), turned to 180 degrees
- moved D3 30.8 mm to (142.8, 67.8), turned to 180 degrees
- moved D4 30.5 mm to (142.8, 66.0), turned to 180 degrees
- moved R4 29.2 mm to (128.0, 76.5)
- moved R3 23.4 mm to (134.0, 73.5)
- moved C4 18.0 mm to (138.0, 72.5), turned to 90 degrees
Routing:
- net Bat: track 6.05 -> 36.4 mm
- net Net-(D3-K): track 0.00 -> 19.8 mm, vias 0 -> 2
- net Net-(D1-K): track 0.00 -> 17.4 mm
- net Net-(R4-Pad2): track 0.00 -> 9.07 mm
- net Net-(D5-A): track 0.00 -> 6.05 mm
- net Vin: track 19.5 -> 25.2 mm
- net GND: track 24.3 -> 28.3 mm
- net Net-(C4-Pad1): track 0.00 -> 2.71 mm
- added copper zone on B.Cu, net GND
- added copper zone on F.Cu, net GND
Other:
- board outline added: 39.5 x 20 mm
